Commit message: add gazebo world. need to calculate the inertia

File: urdf/barista_robot_model.urdf (robot description, URDF)
Before this commit: robot barista_robot, 8 links, 7 joints
Links:
- link base_link: mass None -> 2.0

Commit message: add inertial

File: urdf/barista_robot_model.urdf (robot description, URDF)
Before this commit: robot barista_robot, 8 links, 7 joints
Links:
- link base_link: mass 2.0 -> 17.8
- link base_to_head_rod_1: mass None -> 0.1
- link base_to_head_rod_2: mass None -> 0.1
- link base_to_head_rod_3: mass None -> 0.1
- link base_to_head_rod_4: mass None -> 0.1
- link head_link: mass None -> 10.335
- link left_wheel: mass None -> 1.0
- link right_wheel: mass None -> 1.0

Commit message: rviz urdf completed

File: urdf/barista_robot_model.urdf (robot description, URDF)
Before this commit: robot barista_robot, 8 links, 7 joints
Links:
- added link back_pitch_link; visual sphere radius=0.0352
- added link back_roll_link; visual cylinder length=0.0206 radius=0.0352
- added link back_yaw_link; visual cylinder length=0.0206 radius=0.0352
- added link front_pitch_link; visual sphere radius=0.0352
- added link front_roll_link; visual cylinder length=0.0206 radius=0.0352
- added link front_yaw_link; visual cylinder length=0.0206 radius=0.0352
Joints:
- added joint back_pitch_joint: type continuous, parent back_roll_link, child back_pitch_link, origin xyz=0 0 0 rpy=0 0 0, axis 0 1 0, limit effort=1000.0 velocity=100.0
- added joint back_roll_joint: type continuous, parent back_yaw_link, child back_roll_link, origin xyz=0 0 0 rpy=0 0 0, axis 1 0 0, limit effort=1000.0 velocity=100.0
- added joint back_yaw_joint: type continuous, parent base_link, child back_yaw_link, origin xyz=-0.14 0 -0.075 rpy=0 0 0, axis 0 0 1, limit effort=1000.0 velocity=100.0
- added joint front_pitch_joint: type continuous, parent front_roll_link, child front_pitch_link, origin xyz=0 0 0 rpy=0 0 0, axis 0 1 0, limit effort=1000.0 velocity=100.0
- added joint front_roll_joint: type continuous, parent front_yaw_link, child front_roll_link, origin xyz=0 0 0 rpy=0 0 0, axis 1 0 0, limit effort=1000.0 velocity=100.0
- added joint front_yaw_joint: type continuous, parent base_link, child front_yaw_link, origin xyz=0.14 0 -0.075 rpy=0 0 0, axis 0 0 1, limit effort=1000.0 velocity=100.0

Commit message: working on gazebo

File: urdf/barista_robot_model.urdf (robot description, URDF)
Before this commit: robot barista_robot, 14 links, 13 joints
Links:
- link back_pitch_link: geometry collision sphere radius=0.0352; visual sphere radius=0.0352
- link back_roll_link: geometry collision cylinder length=0.0206 radius=0.0352; visual cylinder length=0.0206 radius=0.0352
- link back_yaw_link: geometry collision cylinder length=0.0206 radius=0.0352; visual cylinder length=0.0206 radius=0.0352
- link base_link: geometry collision cylinder length=0.155 radius=0.178; visual cylinder length=0.155 radius=0.178
- link base_to_head_rod_1: geometry collision cylinder length=0.220 radius=0.010; visual cylinder length=0.220 radius=0.010
- link base_to_head_rod_2: geometry collision cylinder length=0.220 radius=0.010; visual cylinder length=0.220 radius=0.010
- link base_to_head_rod_3: geometry collision cylinder length=0.220 radius=0.010; visual cylinder length=0.220 radius=0.010
- link base_to_head_rod_4: geometry collision cylinder length=0.220 radius=0.010; visual cylinder length=0.220 radius=0.010
- link front_pitch_link: geometry collision sphere radius=0.0352; visual sphere radius=0.0352
- link front_roll_link: geometry collision cylinder length=0.0206 radius=0.0352; visual cylinder length=0.0206 radius=0.0352
- link front_yaw_link: geometry collision cylinder length=0.0206 radius=0.0352; visual cylinder length=0.0206 radius=0.0352
- link head_link: geometry collision cylinder length=0.090 radius=0.178; visual cylinder length=0.090 radius=0.178
- link left_wheel: geometry collision cylinder length=0.0206 radius=0.0352; visual cylinder length=0.0206 radius=0.0352
- link right_wheel: geometry collision cylinder length=0.0206 radius=0.0352; visual cylinder length=0.0206 radius=0.0352

Commit message: gazebo shown successfully

File: urdf/barista_robot_model.urdf (robot description, URDF)
Before this commit: robot barista_robot, 14 links, 13 joints
Links:
- link back_pitch_link: mass None -> 0.001
- link back_roll_link: mass None -> 0.001
- link back_yaw_link: mass None -> 0.001
- link front_pitch_link: mass None -> 0.001
- link front_roll_link: mass None -> 0.001
- link front_yaw_link: mass None -> 0.001

Commit message: Laser success, but not yet visualizable in gazebo

File: urdf/barista_robot_model.urdf (robot description, URDF)
Before this commit: robot barista_robot, 14 links, 13 joints
Links:
- added link laser_scan_frame
- added link laser_scan_link, mass 0.01; collision box size=0.074986 0.074935 0.0408; visual mesh filename=package://barista_robot_description/meshes/rplidar.dae scale=1.0 1.0 1.0
- link back_pitch_link: mass 0.001 -> 0.3
- link back_roll_link: mass 0.001 -> 0.3
- link back_yaw_link: mass 0.001 -> 0.3
- link front_pitch_link: mass 0.001 -> 0.3
- link front_roll_link: mass 0.001 -> 0.3
- link front_yaw_link: mass 0.001 -> 0.3
Joints:
- added joint laser_scan_frame_joint: type fixed, parent laser_scan_link, child laser_scan_frame, origin xyz=0 0 0.03 rpy=0 0 0, axis 0 0 0
- added joint laser_scan_link_joint: type fixed, parent base_link, child laser_scan_link, origin xyz=0.1224 0.0 0.0775 rpy=0 0 0, axis 0 0 1, limit lower=-0.1 upper=0.0 effort=20.0 velocity=2.0

Commit message: laser finished

File: urdf/barista_robot_model.urdf (robot description, URDF)
Before this commit: robot barista_robot, 16 links, 15 joints
Links:
- added link laser_scan_model_link, mass 0.01; collision cylinder length=0.0408 radius=0.037493; visual mesh filename=package://barista_robot_description/meshes/hokuyo_urg_04lx.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 scale=1.0 1.0 1.0
- link laser_scan_link: geometry collision box size=0.02 0.02 0.02; visual box size=0.02 0.02 0.02
Joints:
- added joint laser_scan_model_link_joint: type continuous, parent laser_scan_link, child laser_scan_model_link, origin xyz=0.0 0.0 0.0 rpy=0 0 0, axis 0 0 1, limit effort=10.0 velocity=2.0

Commit message: laser shown completed

File: urdf/barista_robot_model.urdf (robot description, URDF)
Before this commit: robot barista_robot, 17 links, 16 joints
Joints:
- joint laser_scan_frame_joint: origin xyz=0 0 0.03 rpy=0 0 0 -> xyz=0 0 0 rpy=0 0 0

Commit message: part1 tag

File: urdf/barista_robot_model.urdf (robot description, URDF)
Before this commit: robot barista_robot, 17 links, 16 joints
Links:
- link laser_scan_link: geometry collision box size=0.05 0.05 0.05; visual box size=0.02 0.02 0.02
Joints:
- joint laser_scan_frame_joint: origin xyz=0 0 0 rpy=0 0 0 -> xyz=0 0 0.06 rpy=0 0 0

Commit message: part2 finished. submission pressed

File: urdf/barista_robot_model.urdf (robot description, URDF)
Before this commit: robot barista_robot, 17 links, 16 joints
Links:
- link laser_scan_link: geometry collision box size=0.05 0.05 0.05; visual box size=0.05 0.05 0.05

File: urdf/barista_robot_model.urdf.xacro (robot description, xacro)
@@ -12,4 +12,7 @@
 <xacro:property name="wheel_mass" value="1.0"/>
 <xacro:arg name="include_laser" default="true"/>
+<xacro:property name="laser_box_width" value="0.05"/>
+<xacro:property name="laser_box_length" value="0.05"/>
+<xacro:property name="laser_box_height" value="0.05"/>
   <material name="red">
       <color rgba="1.0 0.0 0.0 1"/>
@@ -281,9 +284,10 @@
   <!--if Laser -->
 <xacro:if value="$(arg include_laser)">
-<link name="laser_scan_link">
+<xacro:macro name="laser_scan" params="laser_scan_name">
+<link name="${laser_scan_name}">
     <visual>
       <origin rpy="0 0 0" xyz="0 0 0"/>
       <geometry>
-        <box size="0.02 0.02 0.02"/>
+        <box size="${laser_box_width} ${laser_box_length} ${laser_box_height}"/>
       </geometry>
     </visual>
@@ -291,5 +295,5 @@
        <origin rpy="0 0 0" xyz="0 0 0.0204"/>
       <geometry>
-       <box size="0.05 0.05 0.05"/>
+       <box size="${laser_box_width} ${laser_box_length} ${laser_box_height}"/>
       </geometry>
     </collision>
@@ -300,4 +304,6 @@
     </inertial>
 </link>
+</xacro:macro>
+ <xacro:laser_scan laser_scan_name="laser_scan_link" />
 <joint name="laser_scan_link_joint" type="fixed">
     <origin rpy="0 0 0" xyz="0.1224 0.0 0.0775"/>
@@ -389,7 +395,9 @@
       <joint_name>front_pitch_joint</joint_name>
       <joint_name>back_pitch_joint</joint_name>
+      <xacro:if value="$(arg include_laser)">
       <joint_name>laser_scan_link_joint</joint_name>
       <joint_name>laser_scan_frame_joint</joint_name>
       <joint_name>laser_scan_model_link_joint</joint_name>
+      </xacro:if>
     </plugin>
   </gazebo>

File: urdf/standoff.xacro (robot description, xacro)
@@ -6,5 +6,5 @@
     <origin rpy="0 0 1.5707" xyz="0 0 0.110" />
       <geometry>
-        <cylinder radius="{$rod_radius}" length="{$rod_height}"/>
+        <cylinder radius="${rod_radius}" length="${rod_height}"/>
       </geometry>
     </visual>
@@ -12,5 +12,5 @@
     <origin rpy="0 0 1.5707" xyz="0 0 0.110" />
       <geometry>
-        <cylinder radius="{$rod_radius}" length="{$rod_height}"/>
+        <cylinder radius="${rod_radius}" length="${rod_height}"/>
       </geometry>
     </collision>

Commit message: colorized the robot both rviz and gazebo, change the laser rviz position to laser sensor

File: urdf/barista_robot_model.urdf (robot description, URDF)
Before this commit: robot barista_robot, 17 links, 16 joints
Joints:
- joint laser_scan_link_joint: type fixed -> prismatic

File: urdf/barista_robot_model.urdf.xacro (robot description, xacro)
@@ -41,4 +41,5 @@
       <cylinder radius="${baseheadlink_radius}" length="${baselink_height}"/>
       </geometry>
+                <material name="green_dark"/>
     </visual>
     <collision>
@@ -53,4 +54,7 @@
     </inertial>
   </link>
+  <gazebo reference="base_link">
+    <material>Gazebo/Green</material>
+</gazebo>
   <!-- Standoff Macro -->
   <xacro:include filename="$(find barista_robot_description)/urdf/standoff.xacro" />
@@ -138,4 +142,7 @@
       </inertial>
   </link>
+<gazebo reference="front_yaw_link">
+    <material>Gazebo/Blue</material>
+</gazebo>
   <joint name="front_roll_joint" type="continuous">
     <origin rpy="0 0 0" xyz="0 0 0" />
@@ -197,4 +204,7 @@
       </inertial>
   </link>
+  <gazebo reference="front_pitch_link">
+    <material>Gazebo/Red</material>
+</gazebo>
 <!-- Caster Wheel Back -->
   <joint name="back_yaw_joint" type="continuous">
@@ -226,4 +236,7 @@
       </inertial>
   </link>
+<gazebo reference="back_yaw_link">
+    <material>Gazebo/Blue</material>
+</gazebo>
   <joint name="back_roll_joint" type="continuous">
     <origin rpy="0 0 0" xyz="0 0 0" />
@@ -254,4 +267,7 @@
       </inertial>
   </link>
+<gazebo reference="back_roll_link">
+    <material>Gazebo/Red</material>
+</gazebo>
   <joint name="back_pitch_joint" type="continuous">
     <origin rpy="0 0 0" xyz="0 0 0" />
@@ -282,4 +298,7 @@
       </inertial>
   </link>
+  <gazebo reference="back_pitch_link">
+    <material>Gazebo/Red</material>
+</gazebo>
   <!--if Laser -->
 <xacro:if value="$(arg include_laser)">
@@ -304,7 +323,10 @@
     </inertial>
 </link>
+ <gazebo reference="${laser_scan_name}">
+    <material>Gazebo/Yellow</material>
+</gazebo>
 </xacro:macro>
  <xacro:laser_scan laser_scan_name="laser_scan_link" />
-<joint name="laser_scan_link_joint" type="fixed">
+<joint name="laser_scan_link_joint" type="prismatic">
     <origin rpy="0 0 0" xyz="0.1224 0.0 0.0775"/>
     <parent link="base_link"/>
@@ -342,4 +364,7 @@
     </inertial>
   </link>
+<gazebo reference="laser_scan_model_link_joint">
+    <material>Gazebo/Yellow</material>
+</gazebo>
   <joint name="laser_scan_model_link_joint" type="continuous">
     <origin rpy="0 0 0" xyz="0.0 0.0 0.0"/>
@@ -378,4 +403,5 @@
         </plugin>
     </sensor>
+      <material>Gazebo/Red</material>
 </gazebo>
 </xacro:if>

File: urdf/cup_holder_tray.xacro (robot description, xacro)
@@ -8,4 +8,5 @@
         <cylinder radius="${baseheadlink_radius}" length="${headlink_height}"/>
       </geometry>
+                   <material name="green_dark"/>
     </visual>
    <collision>
@@ -21,4 +22,7 @@
     </inertial>
   </link>
+  <gazebo reference="${cup_holder_tray_name}">
+    <material>Gazebo/Green</material>
+</gazebo>
 </xacro:macro>
 </robot>

File: urdf/standoff.xacro (robot description, xacro)
@@ -8,4 +8,5 @@
         <cylinder radius="${rod_radius}" length="${rod_height}"/>
       </geometry>
+                  <material name="white"/>
     </visual>
     <collision>
@@ -21,4 +22,7 @@
     </inertial>
   </link>
+<gazebo reference="${standoff_name}">
+    <material>Gazebo/Grey</material>
+</gazebo>
   </xacro:macro>
 </robot>

File: urdf/wheel.xacro (robot description, xacro)
@@ -21,4 +21,7 @@
       </inertial>
   </link>
+  <gazebo reference="${wheel_name}">
+    <material>Gazebo/Red</material>
+</gazebo>
 </xacro:macro>
 </robot>
