Commit message: Part 1 finished

File: urdf/barista_robot_model.urdf.xacro (robot description, xacro)
@@ -1,4 +1,7 @@
 <?xml version="1.0"?>
 <robot xmlns:xacro="http://www.ros.org/wiki/xacro" name="barista_robot">
+<xacro:arg name="include_laser" default="true"/>
+<xacro:arg name="robot_name" default=""/>
+<xacro:property name="robot_name" value="$(arg robot_name)"/>
 <xacro:property name="baseheadlink_radius" value="0.178"/>
 <xacro:property name="baselink_height" value="0.155"/>
@@ -11,5 +14,4 @@
 <xacro:property name="wheel_width" value="0.0206"/>
 <xacro:property name="wheel_mass" value="1.0"/>
-<xacro:arg name="include_laser" default="true"/>
 <xacro:property name="laser_box_width" value="0.05"/>
 <xacro:property name="laser_box_length" value="0.05"/>
@@ -397,5 +399,5 @@
         <plugin name="laser" filename="libgazebo_ros_ray_sensor.so">
           <ros>
-            <namespace>/</namespace>
+            <namespace>/${robot_name}</namespace>
             <remapping>~/out:=scan</remapping>
           </ros>
@@ -411,4 +413,5 @@
     <plugin name="barista_robot_joint_state" filename="libgazebo_ros_joint_state_publisher.so">
       <ros>
+          <namespace>/${robot_name}</namespace>
           <remapping>~/out:=joint_states</remapping>
       </ros>
@@ -431,4 +434,8 @@
   <gazebo>
     <plugin filename="libgazebo_ros_diff_drive.so" name="differential_drive_controller">
+        <ros>
+            <namespace>/${robot_name}</namespace>
+            <remapping>/cmd_vel:=cmd_vel</remapping>
+        </ros>
       <!-- wheels -->
       <left_joint>joint_left_wheel</left_joint>
@@ -443,6 +450,9 @@
       <publish_odom>true</publish_odom>
       <publish_odom_tf>true</publish_odom_tf>
-      <odometry_frame>odom</odometry_frame>
-      <robot_base_frame>base_link</robot_base_frame>
+      <!-- TF frames -->
+      <odometry_frame>${robot_name}/odom</odometry_frame>>
+      <robot_base_frame>${robot_name}/base_link</robot_base_frame>
+      <publish_odom_tf>true</publish_odom_tf>
+      <publish_wheel_tf>false</publish_wheel_tf>
     </plugin>
   </gazebo>

Commit message: checkpoint 8, together with robot_chase depository, tf fixed frame to have rick follow morty

File: urdf/barista_robot_model.urdf.xacro (robot description, xacro)
@@ -59,4 +59,12 @@
     <material>Gazebo/Green</material>
 </gazebo>
+ <!-- Attaching TF for TF follow -->
+  <link name="barista_attach_frame">
+  </link>
+  <joint name="barista_attach_frame_joint" type="fixed">
+    <origin rpy="0 0 0" xyz="0.5 0.5 0" />
+    <parent link="base_link" />
+    <child link="barista_attach_frame" />
+  </joint>
   <!-- Standoff Macro -->
   <xacro:include filename="$(find barista_robot_description)/urdf/standoff.xacro" />

Commit message: re-evaulation robot-chase

File: urdf/barista_robot_model.urdf.xacro (robot description, xacro)
@@ -43,5 +43,10 @@
       <cylinder radius="${baseheadlink_radius}" length="${baselink_height}"/>
       </geometry>
+    <xacro:if value="${robot_name == 'morty'}">
                 <material name="green_dark"/>
+    </xacro:if>
+     <xacro:unless value="${robot_name == 'morty'}">
+                <material name="red"/>
+    </xacro:unless>
     </visual>
     <collision>
@@ -56,7 +61,14 @@
     </inertial>
   </link>
-  <gazebo reference="base_link">
-    <material>Gazebo/Green</material>
-</gazebo>
+    <xacro:if value="${robot_name == 'morty'}">
+    <gazebo reference="base_link">
+        <material>Gazebo/Green</material>
+    </gazebo>
+    </xacro:if>
+     <xacro:unless value="${robot_name == 'morty'}">
+    <gazebo reference="base_link">
+        <material>Gazebo/Red</material>
+    </gazebo>
+    </xacro:unless>
  <!-- Attaching TF for TF follow -->
   <link name="barista_attach_frame">
@@ -124,5 +136,5 @@
   </joint>
 <!-- Caster Wheel Front -->
- <joint name="front_yaw_joint" type="continuous">
+ <!--joint name="front_yaw_joint" type="continuous">
     <origin rpy="0 0 0" xyz="0.14 0 -0.075" />
     <parent link="base_link" />
@@ -130,5 +142,5 @@
     <axis xyz="0 0 1" />
     <limit effort="1000.0" velocity="100.0" />
-    <dynamics damping="0.0" friction="0.1"/>
+    <dynamics damping="0.1" friction="0.5"/>
   </joint>
   <link name="front_yaw_link">
@@ -154,6 +166,6 @@
 <gazebo reference="front_yaw_link">
     <material>Gazebo/Blue</material>
-</gazebo>
-  <joint name="front_roll_joint" type="continuous">
+</gazebo-->
+  <!--joint name="front_roll_joint" type="continuous">
     <origin rpy="0 0 0" xyz="0 0 0" />
     <parent link="front_yaw_link" />
@@ -161,5 +173,5 @@
     <axis xyz="1 0 0" />
     <limit effort="1000.0" velocity="100.0" />
-    <dynamics damping="0.0" friction="0.1"/>
+    <dynamics damping="0.1" friction="0.5"/>
   </joint>
   <link name="front_roll_link">
@@ -185,12 +197,12 @@
     <gazebo reference="front_roll_link">
         <material>Gazebo/Red</material>
-    </gazebo>
+    </gazebo-->
   <joint name="front_pitch_joint" type="continuous">
-    <origin rpy="0 0 0" xyz="0 0 0" />
-    <parent link="front_roll_link" />
+    <origin rpy="0 0 0" xyz="0.14 0 -0.075" />
+    <parent link="base_link" />
     <child link="front_pitch_link" />
     <axis xyz="0 1 0" />
     <limit effort="1000.0" velocity="100.0" />
-    <dynamics damping="0.0" friction="0.1"/>
+    <dynamics damping="0.1" friction="0.5"/>
   </joint>
   <link name="front_pitch_link">
@@ -217,10 +229,10 @@
     <kp>1000000000000000000000000000.0</kp>
     <kd>1000000000000000000000000000.0</kd>
-    <mu1>50</mu1>
-    <mu2>50</mu2>
+    <mu1>0.5</mu1>
+    <mu2>0.5</mu2>
     <material>Gazebo/Red</material>
 </gazebo>
 <!-- Caster Wheel Back -->
-  <joint name="back_yaw_joint" type="continuous">
+  <!--joint name="back_yaw_joint" type="continuous">
     <origin rpy="0 0 0" xyz="-0.14 0 -0.075" />
     <parent link="base_link" />
@@ -228,5 +240,5 @@
     <axis xyz="0 0 1" />
     <limit effort="1000.0" velocity="100.0" />
-    <dynamics damping="0.0" friction="0.1"/>
+    <dynamics damping="0.1" friction="0.5"/>
   </joint>
   <link name="back_yaw_link">
@@ -252,6 +264,6 @@
 <gazebo reference="back_yaw_link">
     <material>Gazebo/Blue</material>
-</gazebo>
-  <joint name="back_roll_joint" type="continuous">
+</gazebo-->
+  <!--joint name="back_roll_joint" type="continuous">
     <origin rpy="0 0 0" xyz="0 0 0" />
     <parent link="back_yaw_link" />
@@ -259,5 +271,5 @@
     <axis xyz="1 0 0" />
     <limit effort="1000.0" velocity="100.0" />
-    <dynamics damping="0.0" friction="0.1"/>
+    <dynamics damping="0.1" friction="0.5"/>
   </joint>
   <link name="back_roll_link">
@@ -283,12 +295,12 @@
 <gazebo reference="back_roll_link">
     <material>Gazebo/Red</material>
-</gazebo>
+</gazebo-->
   <joint name="back_pitch_joint" type="continuous">
-    <origin rpy="0 0 0" xyz="0 0 0" />
-    <parent link="back_roll_link" />
+    <origin rpy="0 0 0" xyz="-0.14 0 -0.075" />
+    <parent link="base_link" />
     <child link="back_pitch_link" />
     <axis xyz="0 1 0" />
     <limit effort="1000.0" velocity="100.0" />
-    <dynamics damping="0.0" friction="0.1"/>
+    <dynamics damping="0.1" friction="0.5"/>
   </joint>
   <link name="back_pitch_link">
@@ -315,6 +327,6 @@
     <kp>1000000000000000000000000000.0</kp>
     <kd>1000000000000000000000000000.0</kd>
-    <mu1>50</mu1>
-    <mu2>50</mu2>
+    <mu1>0.5</mu1>
+    <mu2>0.5</mu2>
     <material>Gazebo/Red</material>
 </gazebo>

File: urdf/cup_holder_tray.xacro (robot description, xacro)
@@ -8,5 +8,10 @@
         <cylinder radius="${baseheadlink_radius}" length="${headlink_height}"/>
       </geometry>
-                   <material name="green_dark"/>
+    <xacro:if value="${robot_name == 'morty'}">
+                <material name="green_dark"/>
+    </xacro:if>
+     <xacro:unless value="${robot_name == 'morty'}">
+                <material name="red"/>
+    </xacro:unless>
     </visual>
    <collision>
@@ -22,7 +27,14 @@
     </inertial>
   </link>
-  <gazebo reference="${cup_holder_tray_name}">
-    <material>Gazebo/Green</material>
-</gazebo>
+    <xacro:if value="${robot_name == 'morty'}">
+    <gazebo reference="${cup_holder_tray_name}">
+        <material>Gazebo/Green</material>
+    </gazebo>
+    </xacro:if>
+    <xacro:unless value="${robot_name == 'morty'}">
+        <gazebo reference="${cup_holder_tray_name}">
+        <material>Gazebo/Red</material>
+    </gazebo>
+    </xacro:unless>
 </xacro:macro>
 </robot>

File: urdf/wheel.xacro (robot description, xacro)
@@ -22,8 +22,8 @@
   </link>
   <gazebo reference="${wheel_name}">
-    <kp>1000000000000000000000000.0</kp>
-    <kd>1000000000000000000000000.0</kd>
-    <mu1>1000.0</mu1>
-    <mu2>1000.0</mu2>
+    <kp>1000000000000000000000000000.0</kp>
+    <kd>1000000000000000000000000000.0</kd>
+    <mu1>0.5</mu1>
+    <mu2>0.5</mu2>
     <material>Gazebo/Red</material>
 </gazebo>
